Commit message: Added simulation launch file + xacro script
Added a launch file to make launching gazebo simulation w/ the current robot xacro file simple.

Added a xacro bash script to ease converting the xacro file into a urdf through the launch file.

File: src/amber_sim/urdf/test.urdf (robot description, URDF)
Before this commit: robot AMBER, 3 links, 2 joints
Links:
- added link lower_leg 1, mass 0.21931466; collision box size=0.0356 0.05 0.202; visual mesh filename=package://amber_sim/stl/LOWLEG.stl
- added link lower_leg 2, mass 0.21931466; collision box size=0.0356 0.05 0.202; visual mesh filename=package://amber_sim/stl/LOWLEG.stl
- added link lower_leg 3, mass 0.21931466; collision box size=0.0356 0.05 0.202; visual mesh filename=package://amber_sim/stl/LOWLEG.stl
- added link upper_leg 1, mass 0.29302326; collision box size=0.0356 0.05 0.317; visual mesh filename=package://amber_sim/stl/UPLEG.stl
- added link upper_leg 2, mass 0.29302326; collision box size=0.0356 0.05 0.317; visual mesh filename=package://amber_sim/stl/UPLEG.stl
- added link upper_leg 3, mass 0.29302326; collision box size=0.0356 0.05 0.317; visual mesh filename=package://amber_sim/stl/UPLEG.stl
- link head: geometry visual box size=2 2 0.5
Joints:
- added joint hip_joint 1: type revolute, parent head, child upper_leg 1, origin xyz=0 0 0.123 rpy=0 0 0, axis 0 1 0, limit lower=-1.57079632679 upper=1.57079632679 effort=30.0 velocity=5.0
- added joint hip_joint 2: type revolute, parent head, child upper_leg 2, origin xyz=0 0 0.123 rpy=0 0 0, axis 0 1 0, limit lower=-1.57079632679 upper=1.57079632679 effort=30.0 velocity=5.0
- added joint hip_joint 3: type revolute, parent head, child upper_leg 3, origin xyz=0 0 0.123 rpy=0 0 0, axis 0 1 0, limit lower=-1.57079632679 upper=1.57079632679 effort=30.0 velocity=5.0
- added joint knee_joint 1: type revolute, parent upper_leg 1, child lower_leg 1, axis 0 1 0, limit lower=-1.57079632679 upper=1.57079632679 effort=30.0 velocity=5.0
- added joint knee_joint 2: type revolute, parent upper_leg 2, child lower_leg 2, axis 0 1 0, limit lower=-1.57079632679 upper=1.57079632679 effort=30.0 velocity=5.0
- added joint knee_joint 3: type revolute, parent upper_leg 3, child lower_leg 3, axis 0 1 0, limit lower=-1.57079632679 upper=1.57079632679 effort=30.0 velocity=5.0
