Commit message: Fixed Leg Angle Calculation + Cleaned up file

File: src/amber_sim/urdf/single_leg.xacro (robot description, xacro)
@@ -1,40 +1,25 @@
 <?xml version="1.0" ?>
 <robot name="AMBER_Leg" xmlns:xacro="http://www.ros.org/wiki/xacro">
-  <xacro:property name="to_rad" value="${pi/180}"/>
-  <xacro:property name="arm_angle" value="${75 * to_rad}"/>
-  <xacro:property name="alpha" value="${0.751 * sin(arm_angle)}"/>
-  <xacro:property name="beta" value="${0.751 * cos(arm_angle)}"/>
-<!--
-  <link name="hip_module">
-    <visual>
-      <origin rpy="0 0 0" xyz="0 0 0.0615"/>
-      <geometry>
-        <box size="0.0402 0.05 0.123"/>
-      </geometry>
-      <material name="omni/Blue"/>
-    </visual>
-    <collision>
-      <origin rpy="0 0 0" xyz="0 0 0.0615"/>
-      <geometry>
-        <box size="0.0402 0.05 0.123"/>
-      </geometry>
-    </collision>
-    <inertial>
-      <origin rpy="0 0 0" xyz="0 0 0.0615"/>
-      <mass value="0.190421352"/>
-      <inertia ixx="0.000279744834534" ixy="0" ixz="0" iyy="0.000265717763008" iyz="0" izz="6.53151584738e-05"/>
-    </inertial>
-  </link>
--->
+  <xacro:property name="upper_arm_angle" value="50" />
+  <xacro:property name="TO_RAD" value="${pi/180}"/>
+  <xacro:property name="ANGLEu" value="${upper_arm_angle * TO_RAD}"/>
+  <!-- LOWER LEG DIMENSIONS -->
+  <xacro:property name="xu" value="1" />
+  <xacro:property name="yu" value="0.27" />
+  <xacro:property name="zu" value="0.221" />
+  <!-- UPPER LEG DIMENSIONS -->
+  <xacro:property name="xl" value="0.751" />
+  <xacro:property name="yl" value="0.137" />
+  <xacro:property name="zl" value="0.123" />
+  <!-- Lower Leg Shift -->
+  <xacro:property name="Ju" value="${xl * (2/5)}" /> <!-- Lower Leg Joint Shift -->
+  <xacro:property name="xt" value="${Ju * cos(ANGLEu)}" /> <!-- LLJS Angle X-Shift -->
+  <xacro:property name="zt" value="${Ju * sin(ANGLEu)}" /> <!-- LLJS Angle Z-Shift -->
   <xacro:macro name="amber_leg" params="id x y z joint">
-  <!--
-    <origin rpy = "0 0 0" xyz = "${x} ${y} ${z}"/>
-  -->
   <!-- UPPER LEG -->
     <link name="upper_leg ${id}">
       <visual>
-        <origin rpy="0 ${arm_angle} 0" xyz="${x} ${y} ${z}"/>
+        <origin rpy="0 ${ANGLEu} 0" xyz="${x} ${y} ${z}"/>
         <geometry>
-          <!-- <box size="0.0356 0.05 0.317"/> -->
           <mesh filename="package://amber_sim/stl/UPLEG.stl"/>
         </geometry>
@@ -63,7 +48,6 @@
     <link name="lower_leg ${id}">
       <visual>
-        <origin rpy="0 0 0" xyz="${(0.5 * alpha) + 0.05 + x} ${-0.15 + y} ${-(1.5 * beta) + z}"/>
+        <origin rpy="0 0 0" xyz="${x + xt + 0.3} ${y - 0.15} ${z - zt - 0.03}"/>
         <geometry>
-          <!-- <box size="0.0356 0.05 0.202"/> -->
           <mesh filename="package://amber_sim/stl/LOWLEG.stl"/>
         </geometry>

Commit message: Changed property names + Changed joint params
xdu, ydu, zdu - Upper Leg Dimensions
xdl, ydl, zdl - Lower Leg Dimensions

xpu, ypu, zpu - Upper Leg Position
xpl, ypl, zpl - Lower Leg Position (in terms of hip_joint)

File: src/amber_sim/urdf/single_leg.xacro (robot description, xacro)
@@ -5,20 +5,28 @@
   <xacro:property name="ANGLEu" value="${upper_arm_angle * TO_RAD}"/>
   <!-- LOWER LEG DIMENSIONS -->
-  <xacro:property name="xu" value="1" />
-  <xacro:property name="yu" value="0.27" />
-  <xacro:property name="zu" value="0.221" />
+  <xacro:property name="xdu" value="1" />
+  <xacro:property name="ydu" value="0.27" />
+  <xacro:property name="zdu" value="0.221" />
   <!-- UPPER LEG DIMENSIONS -->
-  <xacro:property name="xl" value="0.751" />
-  <xacro:property name="yl" value="0.137" />
-  <xacro:property name="zl" value="0.123" />
+  <xacro:property name="xdl" value="0.751" />
+  <xacro:property name="ydl" value="0.137" />
+  <xacro:property name="zdl" value="0.123" />
   <!-- Lower Leg Shift -->
-  <xacro:property name="Ju" value="${xl * (2/5)}" /> <!-- Lower Leg Joint Shift -->
+  <xacro:property name="Ju" value="${xdl * (2/5)}" /> <!-- Lower Leg Joint Shift -->
   <xacro:property name="xt" value="${Ju * cos(ANGLEu)}" /> <!-- LLJS Angle X-Shift -->
   <xacro:property name="zt" value="${Ju * sin(ANGLEu)}" /> <!-- LLJS Angle Z-Shift -->
   <xacro:macro name="amber_leg" params="id x y z joint dir">
+    <!-- LOWER LEG POSITION -->
+    <xacro:property name="xpl" value="${0.333}" />
+    <xacro:property name="ypl" value="${y - 0.15*dir}" />
+    <xacro:property name="zpl" value="${.03}" />
+    <!-- UPPER LEG POSITION -->
+    <xacro:property name="xpu" value="${x}" />
+    <xacro:property name="ypu" value="${y}" />
+    <xacro:property name="zpu" value="${z}" />
   <!-- UPPER LEG -->
     <link name="upper_leg ${id}">
       <visual>
-        <origin rpy="0 ${ANGLEu} 0" xyz="${x} ${y} ${z}"/>
+        <origin rpy="0 ${ANGLEu} 0" xyz="${xpu} ${ypu} ${zpu}"/>
         <geometry>
           <mesh filename="package://amber_sim/stl/UPLEG.stl" />
@@ -26,7 +34,7 @@
       </visual>
       <collision>
-        <origin rpy="0 0 0" xyz="0 0 0.1585"/>
+        <origin rpy="0 ${ANGLEu} 0" xyz="${xpu} ${ypu} ${zpu}"/>
         <geometry>
-          <box size="0.0356 0.05 0.317"/>
+          <box size="${xdl} ${ydl} ${zdl}"/>
         </geometry>
       </collision>
@@ -41,6 +49,6 @@
       <child link="lower_leg ${id}"/>
       <dynamics damping="3.0" friction="0.3"/>
-      <limit effort="30.0" lower="-1.57079632679" upper="1.57079632679" velocity="5.0"/>
-      <!-- <origin rpy="0 0 0" xyz="0 0 0.317"/> -->
+      <limit effort="30.0" lower="${-pi/2}" upper="${pi/2}" velocity="5.0"/>
+      <origin rpy="0 0 0" xyz="${x + xt} 0 ${z - zt}"/>
       <axis xyz="0 1 0"/>
     </joint>
@@ -48,5 +56,5 @@
     <link name="lower_leg ${id}">
       <visual>
-        <origin rpy="0 0 0" xyz="${x + xt + 0.3} ${y - 0.15*dir} ${z - zt - 0.03}"/>
+        <origin rpy="0 0 0" xyz="${xpl} ${ypl} ${zpl}"/>
         <geometry>
           <mesh filename="package://amber_sim/stl/LOWLEG.stl" scale="1 ${dir} 1"/>
@@ -54,7 +62,7 @@
       </visual>
       <collision>
-        <origin rpy="0 0 0" xyz="0 0 0.101"/>
+        <origin rpy="0 0 0" xyz="${xpl} ${ypl} ${zpl}"/>
         <geometry>
-          <box size="0.0356 0.05 0.202"/>
+          <box size="${xdl} ${ydl} ${zdl}"/>
         </geometry>
       </collision>
@@ -65,5 +73,5 @@
       </inertial>
     </link>
-    <joint name="hip_joint ${id}" type="revolute">
+    <joint name="hip_joint ${id}" type="fixed">
       <parent link="${joint}"/>
       <child link="upper_leg ${id}"/>
@@ -74,6 +82,4 @@
   </joint>
   </xacro:macro>
-  <!--
   <xacro:amber_leg id="0" x="0" y="0" z="1" joint="head" dir="1"/>
-  -->
 </robot>

Commit message: Added mass & inertia values from fusion360

File: src/amber_sim/urdf/single_leg.xacro (robot description, xacro)
@@ -18,15 +18,17 @@
   <xacro:macro name="amber_leg" params="id x y z joint dir">
     <!-- LOWER LEG POSITION -->
-    <xacro:property name="xpl" value="${0.333}" />
+    <xacro:property name="xpl" value="${0.3}" />
     <xacro:property name="ypl" value="${y - 0.15*dir}" />
     <xacro:property name="zpl" value="${.03}" />
+    <xacro:property name="xyzu" value="${xpu} ${ypu} ${zpu}" />
     <!-- UPPER LEG POSITION -->
     <xacro:property name="xpu" value="${x}" />
     <xacro:property name="ypu" value="${y}" />
     <xacro:property name="zpu" value="${z}" />
+    <xacro:property name="xyzl" value="${xpl} ${ypl} ${zpl}" />
   <!-- UPPER LEG -->
     <link name="upper_leg ${id}">
       <visual>
-        <origin rpy="0 ${ANGLEu} 0" xyz="${xpu} ${ypu} ${zpu}"/>
+        <origin rpy="0 ${ANGLEu} 0" xyz="${xyzu}"/>
         <geometry>
           <mesh filename="package://amber_sim/stl/UPLEG.stl" />
@@ -34,5 +36,5 @@
       </visual>
       <collision>
-        <origin rpy="0 ${ANGLEu} 0" xyz="${xpu} ${ypu} ${zpu}"/>
+        <origin rpy="0 ${ANGLEu} 0" xyz="${xyzu}"/>
         <geometry>
           <box size="${xdl} ${ydl} ${zdl}"/>
@@ -40,14 +42,14 @@
       </collision>
       <inertial>
-        <origin rpy="0 0 0" xyz="0 0 0.1585"/>
-        <mass value="0.29302326"/>
-        <inertia ixx="0.00251484771035" ixy="0" ixz="0" iyy="0.00248474836108" iyz="0" izz="9.19936757328e-05"/>
+        <origin rpy="0 ${ANGLEu} 0" xyz="${xyzu}"/>
+        <mass value="1.624271"/>
+        <inertia ixx="89413.852" ixy="6.821e-10" ixz="30343.48"
+                 iyy="99736.006" iyz="-1.705e-09" izz="17089.95"/>
       </inertial>
     </link>
-    <joint name="knee_joint ${id}" type="revolute">
+    <joint name="knee_joint ${id}" type="continuous">
       <parent link="upper_leg ${id}"/>
       <child link="lower_leg ${id}"/>
-      <dynamics damping="3.0" friction="0.3"/>
-      <limit effort="30.0" lower="${-pi/2}" upper="${pi/2}" velocity="5.0"/>
+      <dynamics damping=".1" friction="0.1"/>
       <origin rpy="0 0 0" xyz="${x + xt} 0 ${z - zt}"/>
       <axis xyz="0 1 0"/>
@@ -56,5 +58,5 @@
     <link name="lower_leg ${id}">
       <visual>
-        <origin rpy="0 0 0" xyz="${xpl} ${ypl} ${zpl}"/>
+        <origin rpy="0 0 0" xyz="${xyzl}"/>
         <geometry>
           <mesh filename="package://amber_sim/stl/LOWLEG.stl" scale="1 ${dir} 1"/>
@@ -62,5 +64,5 @@
       </visual>
       <collision>
-        <origin rpy="0 0 0" xyz="${xpl} ${ypl} ${zpl}"/>
+        <origin rpy="0 0 0" xyz="${xyzl}"/>
         <geometry>
           <box size="${xdl} ${ydl} ${zdl}"/>
@@ -68,7 +70,8 @@
       </collision>
       <inertial>
-        <origin rpy="0 0 0" xyz="0 0 0.101"/>
-        <mass value="0.21931466"/>
-        <inertia ixx="0.000791433503053" ixy="0" ixz="0" iyy="0.000768905501178" iyz="0" izz="6.88531064581e-05"/>
+        <origin rpy="0 0 0" xyz="${xyzl}"/>
+        <mass value="3.442209"/>
+        <inertia ixx="32621.012" ixy="6974.557" ixz="5690.275"
+                 iyy="3.402e+05" iyz="-483.578" izz="3.343e+05"/>
       </inertial>
     </link>
