Commit message: made basis of amber robot xacro

File: src/amber_sim/urdf/amber.xacro (robot description, xacro)
@@ -2,4 +2,20 @@
 <robot name="AMBER" xmlns:xacro="http://www.ros.org/wiki/xacro">
     <xacro:include filename="$(find amber_sim)/urdf/single_leg.xacro"/>
-    <xacro:amber_leg x="0" y="0" z="1"/>
+    <link name="head">
+    <visual>
+      <origin rpy="0 0 0" xyz="0.7 1 1.5"/>
+      <geometry>
+        <box size="2 2 0.5"/>
+      </geometry>
+    </visual>
+    <inertial>
+      <origin rpy="0 0 0" xyz="0 0 0.0615"/>
+      <mass value="0.190421352"/>
+      <inertia ixx="0.000279744834534" ixy="0" ixz="0" iyy="0.000265717763008" iyz="0" izz="6.53151584738e-05"/>
+    </inertial>
+  </link>
+    <xacro:amber_leg id="0" x="0" y="0" z="1" joint="head"/>
+    <xacro:amber_leg id="1" x="0" y="2" z="1" joint="head"/>
+    <xacro:amber_leg id="2" x="1.5" y="0" z="1" joint="head"/>
+    <xacro:amber_leg id="3" x="1.5" y="2" z="1" joint="head"/>
 </robot>

File: src/amber_sim/urdf/single_leg.xacro (robot description, xacro)
@@ -26,19 +26,13 @@
     </inertial>
   </link>
-  <joint name="hip_joint" type="revolute">
-    <parent link="hip_module"/>
-    <child link="upper_leg"/>
-    <dynamics damping="3.0" friction="0.3"/>
-    <limit effort="30.0" lower="-1.57079632679" upper="1.57079632679" velocity="5.0"/>
-    <origin rpy="0 0 0" xyz="0 0 0.123"/>
-    <axis xyz="0 1 0"/>
-  </joint>
 -->
-  <xacro:macro name="amber_leg" params="x y z">
+  <xacro:macro name="amber_leg" params="id x y z joint">
+  <!--
     <origin rpy = "0 0 0" xyz = "${x} ${y} ${z}"/>
+  -->
   <!-- UPPER LEG -->
-    <link name="upper_leg">
+    <link name="upper_leg ${id}">
       <visual>
-        <origin rpy="0 ${arm_angle} 0" xyz="0 0 0"/>
+        <origin rpy="0 ${arm_angle} 0" xyz="${x} ${y} ${z}"/>
         <geometry>
           <!-- <box size="0.0356 0.05 0.317"/> -->
@@ -58,7 +52,7 @@
       </inertial>
     </link>
-    <joint name="knee_joint" type="revolute">
-      <parent link="upper_leg"/>
-      <child link="lower_leg"/>
+    <joint name="knee_joint ${id}" type="revolute">
+      <parent link="upper_leg ${id}"/>
+      <child link="lower_leg ${id}"/>
       <dynamics damping="3.0" friction="0.3"/>
       <limit effort="30.0" lower="-1.57079632679" upper="1.57079632679" velocity="5.0"/>
@@ -67,7 +61,7 @@
     </joint>
   <!-- LOWER LEG -->
-    <link name="lower_leg">
+    <link name="lower_leg ${id}">
       <visual>
-        <origin rpy="0 0 0" xyz="${(0.5 * alpha) + 0.05} -0.15 -${1.5 * beta}"/>
+        <origin rpy="0 0 0" xyz="${(0.5 * alpha) + 0.05 + x} ${-0.15 + y} ${-(1.5 * beta) + z}"/>
         <geometry>
           <!-- <box size="0.0356 0.05 0.202"/> -->
@@ -87,4 +81,12 @@
       </inertial>
     </link>
+    <joint name="hip_joint ${id}" type="revolute">
+      <parent link="${joint}"/>
+      <child link="upper_leg ${id}"/>
+      <dynamics damping="3.0" friction="0.3"/>
+      <limit effort="30.0" lower="-1.57079632679" upper="1.57079632679" velocity="5.0"/>
+      <origin rpy="0 0 0" xyz="0 0 0.123"/>
+      <axis xyz="0 1 0"/>
+  </joint>
   </xacro:macro>
 </robot>

File: src/amber_sim/urdf/test.urdf (robot description, URDF)
Before this commit: robot AMBER, 2 links, 1 joints
Links:
- removed link lower_leg
- removed link upper_leg
- added link head, mass 0.190421352; visual box size=0 0 0
- added link lower_leg 0, mass 0.21931466; collision box size=0.0356 0.05 0.202; visual mesh filename=package://amber_sim/stl/LOWLEG.stl
- added link upper_leg 0, mass 0.29302326; collision box size=0.0356 0.05 0.317; visual mesh filename=package://amber_sim/stl/UPLEG.stl
Joints:
- removed joint knee_joint
- added joint hip_joint 0: type revolute, parent head, child upper_leg 0, origin xyz=0 0 0.123 rpy=0 0 0, axis 0 1 0, limit lower=-1.57079632679 upper=1.57079632679 effort=30.0 velocity=5.0
- added joint knee_joint 0: type revolute, parent upper_leg 0, child lower_leg 0, axis 0 1 0, limit lower=-1.57079632679 upper=1.57079632679 effort=30.0 velocity=5.0

Commit message: Changeable Orientation
Orientation of the leg can be changed using the 'dir' parameter on the amber_leg macro.
dir = 1; right-hand
dir = -1; left-land

File: src/amber_sim/urdf/amber.xacro (robot description, xacro)
@@ -15,7 +15,7 @@
     </inertial>
   </link>
-    <xacro:amber_leg id="0" x="0" y="0" z="1" joint="head"/>
-    <xacro:amber_leg id="1" x="0" y="2" z="1" joint="head"/>
-    <xacro:amber_leg id="2" x="1.5" y="0" z="1" joint="head"/>
-    <xacro:amber_leg id="3" x="1.5" y="2" z="1" joint="head"/>
+    <xacro:amber_leg id="bottom_right" x="0" y="0" z="1" joint="head" dir="1"/>
+    <xacro:amber_leg id="bottom_left" x="0" y="2" z="1" joint="head" dir="-1"/>
+    <xacro:amber_leg id="top_right" x="1.5" y="0" z="1" joint="head" dir="1"/>
+    <xacro:amber_leg id="top_left" x="1.5" y="2" z="1" joint="head" dir="-1"/>
 </robot>

File: src/amber_sim/urdf/single_leg.xacro (robot description, xacro)
@@ -16,5 +16,5 @@
   <xacro:property name="xt" value="${Ju * cos(ANGLEu)}" /> <!-- LLJS Angle X-Shift -->
   <xacro:property name="zt" value="${Ju * sin(ANGLEu)}" /> <!-- LLJS Angle Z-Shift -->
-  <xacro:macro name="amber_leg" params="id x y z joint">
+  <xacro:macro name="amber_leg" params="id x y z joint dir">
   <!-- UPPER LEG -->
     <link name="upper_leg ${id}">
@@ -22,5 +22,5 @@
         <origin rpy="0 ${ANGLEu} 0" xyz="${x} ${y} ${z}"/>
         <geometry>
-          <mesh filename="package://amber_sim/stl/UPLEG.stl"/>
+          <mesh filename="package://amber_sim/stl/UPLEG.stl" />
         </geometry>
       </visual>
@@ -48,7 +48,7 @@
     <link name="lower_leg ${id}">
       <visual>
-        <origin rpy="0 0 0" xyz="${x + xt + 0.3} ${y - 0.15} ${z - zt - 0.03}"/>
+        <origin rpy="0 0 0" xyz="${x + xt + 0.3} ${y - 0.15*dir} ${z - zt - 0.03}"/>
         <geometry>
-          <mesh filename="package://amber_sim/stl/LOWLEG.stl"/>
+          <mesh filename="package://amber_sim/stl/LOWLEG.stl" scale="1 ${dir} 1"/>
         </geometry>
       </visual>
@@ -74,4 +74,6 @@
   </joint>
   </xacro:macro>
-  <xacro:amber_leg id="0" x="0" y="0" z="1" joint="head"/>
+  <!--
+  <xacro:amber_leg id="0" x="0" y="0" z="1" joint="head" dir="1"/>
+  -->
 </robot>

Commit message: Added body model + added mass/inertial properties from fusion360 + added materials to models

File: src/amber_sim/urdf/amber.xacro (robot description, xacro)
@@ -1,19 +1,27 @@
 <?xml version="1.0" ?>
 <robot name="AMBER" xmlns:xacro="http://www.ros.org/wiki/xacro">
+    <!-- BODY DIMENSIONS -->
+    <xacro:property name="xdb" value="1.71" />
+    <xacro:property name="ydb" value="0.683" />
+    <xacro:property name="zdb" value="0.41" />
     <xacro:include filename="$(find amber_sim)/urdf/single_leg.xacro"/>
     <link name="head">
     <visual>
-      <origin rpy="0 0 0" xyz="0.7 1 1.5"/>
+      <origin rpy="0 0 0" xyz="0 0 1"/>
+      <material name="body">
+        <color rgba="0.5 0.6 0.9 1.0" />
+      </material>
       <geometry>
-        <box size="2 2 0.5"/>
+        <mesh filename="package://amber_sim/stl/BODY.stl"/>
       </geometry>
     </visual>
     <inertial>
       <origin rpy="0 0 0" xyz="0 0 0.0615"/>
-      <mass value="0.190421352"/>
-      <inertia ixx="0.000279744834534" ixy="0" ixz="0" iyy="0.000265717763008" iyz="0" izz="6.53151584738e-05"/>
+      <mass value="54.40980"/>
+      <inertia ixx="3.663e+06" ixy="14390.775" ixz="1.424e+06"
+               iyy="1.560e+07" iyz="8027.636" izz="1.721e+07"/>
     </inertial>
   </link>
-    <xacro:amber_leg id="bottom_right" x="0" y="0" z="1" joint="head" dir="1"/>
+    <xacro:amber_leg id="bottom_right" x="${0}" y="${-ydb/2}" z="1" joint="head" dir="1"/>
     <xacro:amber_leg id="bottom_left" x="0" y="2" z="1" joint="head" dir="-1"/>
     <xacro:amber_leg id="top_right" x="1.5" y="0" z="1" joint="head" dir="1"/>

File: src/amber_sim/urdf/single_leg.xacro (robot description, xacro)
@@ -31,4 +31,7 @@
       <visual>
         <origin rpy="0 ${ANGLEu} 0" xyz="${xyzu}"/>
+        <material name="ul">
+          <color rgba="0.6 0.6 0.6 1.0" />
+        </material>
         <geometry>
           <mesh filename="package://amber_sim/stl/UPLEG.stl" />
@@ -59,4 +62,7 @@
       <visual>
         <origin rpy="0 0 0" xyz="${xyzl}"/>
+        <material name="ll">
+          <color rgba="0.6 0.6 0.7 1.0" />
+        </material>
         <geometry>
           <mesh filename="package://amber_sim/stl/LOWLEG.stl" scale="1 ${dir} 1"/>

Commit message: Finished base design of amber.xacro
Numbers used to position the legs in amber.xacro are preliminary.

File: src/amber_sim/urdf/amber.xacro (robot description, xacro)
@@ -23,7 +23,7 @@
     </inertial>
   </link>
-    <xacro:amber_leg id="bottom_right" x="${0}" y="${-ydb/2}" z="1" joint="head" dir="1"/>
-    <xacro:amber_leg id="bottom_left" x="0" y="2" z="1" joint="head" dir="-1"/>
-    <xacro:amber_leg id="top_right" x="1.5" y="0" z="1" joint="head" dir="1"/>
-    <xacro:amber_leg id="top_left" x="1.5" y="2" z="1" joint="head" dir="-1"/>
+    <xacro:amber_leg id="bottom_right" x="${xt-0.6}" y="${-ydb/2 - ydl/2}" z="${1-1.5*zt}" joint="head" dir="1"/>
+    <xacro:amber_leg id="bottom_left" x="${xt-0.6}" y="${ydb/2 + ydl/2}" z="${1-1.5*zt}" joint="head" dir="-1"/>
+    <xacro:amber_leg id="top_right" x="${xt+0.6}" y="${-ydb/2 - ydl/2}" z="${1-1.5*zt}" joint="head" dir="1"/>
+    <xacro:amber_leg id="top_left" x="${xt+0.6}" y="${ydb/2 + ydl/2}" z="${1-1.5*zt}" joint="head" dir="-1"/>
 </robot>

File: src/amber_sim/urdf/single_leg.xacro (robot description, xacro)
@@ -1,5 +1,5 @@
 <?xml version="1.0" ?>
 <robot name="AMBER_Leg" xmlns:xacro="http://www.ros.org/wiki/xacro">
-  <xacro:property name="upper_arm_angle" value="50" />
+  <xacro:property name="upper_arm_angle" value="80" />
   <xacro:property name="TO_RAD" value="${pi/180}"/>
   <xacro:property name="ANGLEu" value="${upper_arm_angle * TO_RAD}"/>
@@ -91,4 +91,6 @@
   </joint>
   </xacro:macro>
+  <!--
   <xacro:amber_leg id="0" x="0" y="0" z="1" joint="head" dir="1"/>
+  -->
 </robot>
